File: ClockDivider/ClockDiv_v2/ClockDiv_v2.kicad_sch (KiCad schematic)
At the start: 39 parts, among them J1 Conn_02x05_Counter_Clockwise, J2 ClockIn, J3 ResetIn, J4 /2, J5 /4, J6 /8, J7 /16, J8 /32, J9 /64, Q1 2N3904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

Commit message: Redesigned PCB
Parts:
- removed C1: 0.1u, Capacitor_THT:CP_Radial_D5.0mm_P2.50mm, symbol Device:C_Polarized
- removed C2: 0.33u, Capacitor_THT:C_Disc_D5.0mm_W2.5mm_P2.50mm, symbol Device:C
- removed C3: 0.1u, Capacitor_THT:C_Disc_D5.0mm_W2.5mm_P2.50mm, symbol Device:C
- removed D7: 1N4148, Diode_THT:D_DO-35_SOD27_P7.62mm_Horizontal, symbol Diode:1N4148
- removed J1: Conn_02x05_Counter_Clockwise, Connector_PinHeader_2.54mm:PinHeader_2x05_P2.54mm_Vertical, symbol Connector_Generic:Conn_02x05_Counter_Clockwise
- removed U2: L7805, Package_TO_SOT_THT:TO-220-3_Horizontal_TabDown, symbol Regulator_Linear:L7805
- added C1: 0.1u, Capacitor_THT:C_Disc_D5.0mm_W2.5mm_P2.50mm, symbol Device:C
- added C2: 10u, Capacitor_THT:CP_Radial_D5.0mm_P2.50mm, symbol Device:C_Polarized
- added J10: Conn_02x08_Odd_Even, Connector_PinHeader_2.54mm:PinHeader_2x08_P2.54mm_Vertical, symbol Connector_Generic:Conn_02x08_Odd_Even
Connections:
- net +12V: now also J10.10 (Pin_10), J10.9 (Pin_9)
- net -12V: now also J10.1 (Pin_1), J10.2 (Pin_2)
- net GND: now also C1.2, C2.2, J10.3 (Pin_3), J10.4 (Pin_4), J10.5 (Pin_5), J10.6 (Pin_6), J10.7 (Pin_7), J10.8 (Pin_8)
- net +5V: now reaches R2.1, U1.16 (VDD)
- net +5V: now also C1.1, C2.1, J10.11 (Pin_11), J10.12 (Pin_12)
- new net: J10.13 (Pin_13), J10.14 (Pin_14)
- new net: J10.15 (Pin_15), J10.16 (Pin_16)
- no-connect marks 6 -> 10
Other:
- note added: "Power input"
- moved on the sheet: D1, D2, D3, D4, D5, D6, J2, J3, J4, J5, J6, J7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
